Commit message: Change base frame offset
Remove the default 180 deg offset from the ur_common URDF.
Makes the configuration in accordance with the UR robot controller.

File: ur_description/urdf/inc/ur_macro.xacro (robot description, xacro)
@@ -55,4 +55,6 @@
     safety_k_position:=20"
   >
+    <!-- Set base frame z-axis rotation here -->
+    <xacro:property name="base_z_rotation" value="0" />
     <!-- Load configuration data from the provided .yaml files -->
     <xacro:read_model_data
@@ -67,5 +69,5 @@
     <link name="${prefix}base_link_inertia">
       <visual>
-        <origin xyz="0 0 0" rpy="0 0 ${pi}"/>
+        <origin xyz="0 0 0" rpy="0 0 ${base_z_rotation}"/>
         <geometry>
           <mesh filename="${base_visual_mesh}"/>
@@ -76,5 +78,5 @@
       </visual>
       <collision>
-        <origin xyz="0 0 0" rpy="0 0 ${pi}"/>
+        <origin xyz="0 0 0" rpy="0 0 ${base_z_rotation}"/>
         <geometry>
           <mesh filename="${base_collision_mesh}"/>
@@ -215,5 +217,5 @@
            link/frame) to introduce the necessary rotation over Z (of pi rad).
       -->
-      <origin xyz="0 0 0" rpy="0 0 ${pi}" />
+      <origin xyz="0 0 0" rpy="0 0 ${base_z_rotation}" />
     </joint>
     <joint name="${prefix}shoulder_pan_joint" type="revolute">
@@ -297,5 +299,5 @@
            the UR controller.
       -->
-      <origin xyz="0 0 0" rpy="0 0 ${pi}"/>
+      <origin xyz="0 0 0" rpy="0 0 ${base_z_rotation}"/>
       <parent link="${prefix}base_link"/>
       <child link="${prefix}base"/>
